File: Buck Converter.kicad_sch (KiCad schematic)
At the start: 15 parts, among them J1 Conn_01x02, J2 Conn_01x02, J3 Conn_01x02, Q1 IRFZ44N, U1 TC4422

Commit message: Created Layout
Signed-off-by: blyons-dev <bthelyons@gmail.com>
Parts:
- C1, C2: footprint (none) -> Capacitor_THT:C_Radial_D10.0mm_H12.5mm_P5.00mm
- D1: footprint (none) -> Diode_THT:D_DO-41_SOD81_P10.16mm_Horizontal
- D2: footprint Package_TO_SOT_SMD:SOT-23 -> Package_TO_SOT_THT:TO-220-3_Vertical
- L1: footprint (none) -> Inductor_THT_Wurth:L_Wurth_WE-HCFT-2012_LeadDiameter1.2mm
Connections:
- net at D2.3 (K), R2.2: now also D1.1 (K), Q1.1 (G)
- now unconnected: D2.2 (A)
